File: biosphereMonitor.brd (EAGLE design)
At the start: 85 x 85 mm, 35 parts, among them IC1 XMEGA32A4AU, IC2 LM35, IC3 FT232RL, Q1 16Mhz, Q2 32kHz

Commit message: added light sensor to schematic
Parts:
- added D1: LM4050 2.5, Tjarks_Bauteile (1):SOT23
- added PH1: BPW 96C TEL, photo-elements:T0-46-A10XX
- added R6: 1k, rcl:R0805
- added R7: 2k2, rcl:R0805
- added R8: 3k3, rcl:R0805
Connections:
- new net 2.5V: D1.1, R6.1, R8.2
- net +5V: now also R6.2
- net GND: now also D1.2, PH1.2, R7.1
- net LIGHT: now also PH1.1, R7.2, R8.1
Changed lines of the file:
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@@
 <attribute name="VALUE" x="-10.09" y="-3.175" locked="yes" size="1.27" layer="27"/>
+</element>
+<element name="D1" library="Tjarks_Bauteile (1)" package="SOT23" value="LM4050 2.5" x="56.32" y="2.56" smashed="yes">
+<attribute name="NAME" x="54.415" y="4.465" size="1.27" layer="25"/>
+<attribute name="VALUE" x="54.415" y="-0.615" size="1.27" layer="27"/>
+</element>
+<element name="R6" library="rcl" library_urn="urn:adsk.eagle:library:334" package="R0805" package3d_urn="urn:adsk.eagle:package:23553/2" value="1k" x="60.16" y="10.24" smashed="yes">
+<attribute name="NAME" x="59.525" y="11.51" size="1.27" layer="25"/>
+<attribute name="POPULARITY" value="86" x="60.16" y="10.24" size="1.778" layer="27" display="off"/>
+<attribute name="SPICEPREFIX" value="R" x="60.16" y="10.24" size="1.778" layer="27" display="off"/>
+<attribute name="VALUE" x="59.525" y="7.7" size="1.27" layer="27"/>
+</element>
+<element name="PH1" library="photo-elements" library_urn="urn:adsk.eagle:library:323" package="T0-46-A10XX" package3d_urn="urn:adsk.eagle:package:22201/1" value="BPW 96C TEL" x="38.4" y="0" smashed="yes" rot="R90">
+<attribute name="NAME" x="33.24" y="-1.905" size="1.27" layer="25" rot="R90"/>
+<attribute name="POPULARITY" value="0" x="38.4" y="0" size="1.778" layer="27" rot="R90" display="off"/>
+<attribute name="VALUE" x="34.59" y="-1.905" size="1.27" layer="27" rot="R90"/>
+</element>
+<element name="R7" library="rcl" library_urn="urn:adsk.eagle:library:334" package="R0805" package3d_urn="urn:adsk.eagle:package:23553/2" value="2k2" x="52.48" y="10.24" smashed="yes">
+<attribute name="NAME" x="51.845" y="11.51" size="1.27" layer="25"/>
+<attribute name="POPULARITY" value="86" x="52.48" y="10.24" size="1.778" layer="27" display="off"/>
+<attribute name="SPICEPREFIX" value="R" x="52.48" y="10.24" size="1.778" layer="27" display="off"/>
+<attribute name="VALUE" x="51.845" y="7.7" size="1.27" layer="27"/>
+</element>
+<element name="R8" library="rcl" library_urn="urn:adsk.eagle:library:334" package="R0805" package3d_urn="urn:adsk.eagle:package:23553/2" value="3k3" x="57.6" y="16.64" smashed="yes">
+<attribute name="NAME" x="56.965" y="17.91" size="1.27" layer="25"/>
+<attribute name="POPULARITY" value="86" x="57.6" y="16.64" size="1.778" layer="27" display="off"/>
+<attribute name="SPICEPREFIX" value="R" x="57.6" y="16.64" size="1.778" layer="27" display="off"/>
+<attribute name="VALUE" x="56.965" y="14.1" size="1.27" layer="27"/>
 </element>
 </elements>
@@
 <vertex x="26.88" y="-14.08"/>
 </polygon>
-<wire x1="-91.71" y1="39.37" x2="-98.06" y2="39.37" width="0" layer="19" extent="1-1"/>
-<wire x1="-85.36" y1="39.37" x2="-91.71" y2="39.37" width="0" layer="19" extent="1-1"/>
-<wire x1="-79.01" y1="39.37" x2="-85.36" y2="39.37" width="0" layer="19" extent="1-1"/>
-<wire x1="-98.06" y1="48.26" x2="-98.06" y2="39.37" width="0" layer="19" extent="1-1"/>
-<wire x1="-91.71" y1="48.26" x2="-98.06" y2="48.26" width="0" layer="19" extent="1-1"/>
-<wire x1="-85.36" y1="48.26" x2="-91.71" y2="48.26" width="0" layer="19" extent="1-1"/>
-<wire x1="-79.01" y1="48.26" x2="-85.36" y2="48.26" width="0" layer="19" extent="1-1"/>
-<wire x1="-72.66" y1="48.26" x2="-79.01" y2="48.26" width="0" layer="19" extent="1-1"/>
-<wire x1="-66.31" y1="48.26" x2="-72.66" y2="48.26" width="0" layer="19" extent="1-1"/>
-<wire x1="-59.96" y1="48.26" x2="-66.31" y2="48.26" width="0" layer="19" extent="1-1"/>
-<wire x1="-59.96" y1="54.61" x2="-59.96" y2="48.26" width="0" layer="19" extent="1-1"/>
-<wire x1="-80.6" y1="59.69" x2="-79.01" y2="48.26" width="0" layer="19" extent="1-1"/>
-<wire x1="-31.99" y1="5.08" x2="-59.96" y2="48.26" width="0" layer="19" extent="1-1"/>
-<wire x1="-31.99" y1="2.54" x2="-31.99" y2="5.08" width="0" layer="19" extent="1-1"/>
-<wire x1="-31.99" y1="0" x2="-31.99" y2="2.54" width="0" layer="19" extent="1-1"/>
-<wire x1="-31.99" y1="-2.54" x2="-31.99" y2="0" width="0" layer="19" extent="1-1"/>
+<contactref element="D1" pad="2"/>
+<contactref element="R7" pad="1"/>
+<contactref element="PH1" pad="2"/>
+<wire x1="38.4" y1="1.7" x2="51.53" y2="10.24" width="0" layer="19" extent="1-1"/>
+<wire x1="57.27" y1="1.46" x2="38.4" y2="1.7" width="0" layer="19" extent="1-1"/>
+<wire x1="-31.99" y1="-2.54" x2="57.27" y2="1.46" width="0" layer="19" extent="1-1"/>
+<wire x1="-31.99" y1="0" x2="-31.99" y2="-2.54" width="0" layer="19" extent="1-1"/>
+<wire x1="-31.99" y1="2.54" x2="-31.99" y2="0" width="0" layer="19" extent="1-1"/>
+<wire x1="-31.99" y1="5.08" x2="-31.99" y2="2.54" width="0" layer="19" extent="1-1"/>
 <wire x1="-7.12" y1="16.24" x2="-31.99" y2="5.08" width="0" layer="19" extent="1-1"/>
 <wire x1="-0.52" y1="12.04" x2="-7.12" y2="16.24" width="0" layer="19" extent="1-1"/>
@@
 <wire x1="4.45" y1="-39.08" x2="4.45" y2="-33.18" width="0" layer="19" extent="1-1"/>
 <wire x1="-12.914" y1="-27.31" x2="-3.425" y2="-25.805" width="0" layer="19" extent="1-1"/>
+<wire x1="-59.96" y1="48.26" x2="-31.99" y2="5.08" width="0" layer="19" extent="1-1"/>
+<wire x1="-66.31" y1="48.26" x2="-59.96" y2="48.26" width="0" layer="19" extent="1-1"/>
+<wire x1="-72.66" y1="48.26" x2="-66.31" y2="48.26" width="0" layer="19" extent="1-1"/>
+<wire x1="-79.01" y1="48.26" x2="-72.66" y2="48.26" width="0" layer="19" extent="1-1"/>
+<wire x1="-85.36" y1="48.26" x2="-79.01" y2="48.26" width="0" layer="19" extent="1-1"/>
+<wire x1="-91.71" y1="48.26" x2="-85.36" y2="48.26" width="0" layer="19" extent="1-1"/>
+<wire x1="-98.06" y1="48.26" x2="-91.71" y2="48.26" width="0" layer="19" extent="1-1"/>
+<wire x1="-59.96" y1="54.61" x2="-59.96" y2="48.26" width="0" layer="19" extent="1-1"/>
+<wire x1="-98.06" y1="39.37" x2="-98.06" y2="48.26" width="0" layer="19" extent="1-1"/>
+<wire x1="-91.71" y1="39.37" x2="-98.06" y2="39.37" width="0" layer="19" extent="1-1"/>
+<wire x1="-85.36" y1="39.37" x2="-91.71" y2="39.37" width="0" layer="19" extent="1-1"/>
+<wire x1="-79.01" y1="39.37" x2="-85.36" y2="39.37" width="0" layer="19" extent="1-1"/>
+<wire x1="-80.6" y1="59.69" x2="-79.01" y2="48.26" width="0" layer="19" extent="1-1"/>
 </signal>
 <signal name="N$1">
@@
 <signal name="LIGHT">
 <contactref element="IC1" pad="41"/>
+<contactref element="PH1" pad="1"/>
+<contactref element="R7" pad="2"/>
+<contactref element="R8" pad="1"/>
+<wire x1="53.43" y1="10.24" x2="56.65" y2="16.64" width="0" layer="19" extent="1-1"/>
+<wire x1="38.4" y1="-1.7" x2="53.43" y2="10.24" width="0" layer="19" extent="1-1"/>
+<wire x1="-2.92" y1="23.64" x2="38.4" y2="-1.7" width="0" layer="19" extent="1-1"/>
 </signal>
 <signal name="SOIL">
@@
 <wire x1="25.6" y1="-12.78" x2="23.3648" y2="-10.5448" width="0.1524" layer="1"/>
 <wire x1="23.3648" y1="-10.5448" x2="17.024" y2="-10.5448" width="0.1524" layer="1"/>
+<contactref element="R6" pad="2"/>
+<wire x1="-14.946" y1="-27.31" x2="61.11" y2="10.24" width="0" layer="19" extent="1-1"/>
 <wire x1="-3.425" y1="-21.905" x2="-14.946" y2="-27.31" width="0" layer="19" extent="1-1"/>
 <wire x1="-6.28" y1="0" x2="-3.425" y2="-21.905" width="0" layer="19" extent="1-1"/>
@@
 <via x="38.4" y="-11.52" extent="1-16" drill="0.35"/>
 </signal>
+<signal name="2.5V">
+<contactref element="D1" pad="1"/>
+<contactref element="R6" pad="1"/>
+<contactref element="R8" pad="2"/>
+<wire x1="59.21" y1="10.24" x2="58.55" y2="16.64" width="0" layer="19" extent="1-1"/>
+<wire x1="55.37" y1="1.46" x2="59.21" y2="10.24" width="0" layer="19" extent="1-1"/>
+</signal>
 </signals>

Commit message: added reference in schematic
Connections:
- net 2.5V: now also IC1.40
- net T_OUT: now also IC1.43; no longer IC1.40
Changed lines of the file:
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@@
 </signal>
 <signal name="T_OUT">
-<contactref element="IC1" pad="40"/>
 <contactref element="IC2" pad="C"/>
 <contactref element="C5" pad="2"/>
 <contactref element="TP6" pad="TP"/>
 <wire x1="29.44" y1="-10.24" x2="16.64" y2="-10.24" width="0.1524" layer="1"/>
+<contactref element="IC1" pad="43"/>
 <wire x1="-58.06" y1="48.26" x2="-95.84" y2="59.69" width="0" layer="19" extent="1-1"/>
-<wire x1="-2.12" y1="23.64" x2="-58.06" y2="48.26" width="0" layer="19" extent="1-1"/>
-<wire x1="16.64" y1="-10.24" x2="-2.12" y2="23.64" width="0" layer="19" extent="1-1"/>
+<wire x1="-4.52" y1="23.64" x2="-58.06" y2="48.26" width="0" layer="19" extent="1-1"/>
+<wire x1="16.64" y1="-10.24" x2="-4.52" y2="23.64" width="0" layer="19" extent="1-1"/>
 </signal>
 <signal name="USB_RX">
@@
 <contactref element="R6" pad="1"/>
 <contactref element="R8" pad="2"/>
+<contactref element="IC1" pad="40"/>
 <wire x1="59.21" y1="10.24" x2="58.55" y2="16.64" width="0" layer="19" extent="1-1"/>
 <wire x1="55.37" y1="1.46" x2="59.21" y2="10.24" width="0" layer="19" extent="1-1"/>
+<wire x1="-2.12" y1="23.64" x2="58.55" y2="16.64" width="0" layer="19" extent="1-1"/>
 </signal>
 </signals>

Commit message: ups
Parts:
- added R10: 3k3, rcl:R0805
- added R9: 2k2, rcl:R0805
Connections:
- new net 1V: IC1.40, R10.1, R9.2
- net 2.5V: now also R10.2; no longer IC1.40
- net GND: now also R9.1
Changed lines of the file:
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@@
 <attribute name="VALUE" x="56.965" y="14.1" size="1.27" layer="27"/>
+</element>
+<element name="R9" library="rcl" library_urn="urn:adsk.eagle:library:334" package="R0805" package3d_urn="urn:adsk.eagle:package:23553/2" value="2k2" x="-65.28" y="8.96" smashed="yes">
+<attribute name="NAME" x="-65.915" y="10.23" size="1.27" layer="25"/>
+<attribute name="POPULARITY" value="86" x="-65.28" y="15.36" size="1.778" layer="27" display="off"/>
+<attribute name="SPICEPREFIX" value="R" x="-65.28" y="15.36" size="1.778" layer="27" display="off"/>
+<attribute name="VALUE" x="-65.915" y="6.42" size="1.27" layer="27"/>
+</element>
+<element name="R10" library="rcl" library_urn="urn:adsk.eagle:library:334" package="R0805" package3d_urn="urn:adsk.eagle:package:23553/2" value="3k3" x="-65.28" y="14.08" smashed="yes">
+<attribute name="NAME" x="-65.915" y="15.35" size="1.27" layer="25"/>
+<attribute name="POPULARITY" value="86" x="-65.28" y="7.68" size="1.778" layer="27" display="off"/>
+<attribute name="SPICEPREFIX" value="R" x="-65.28" y="7.68" size="1.778" layer="27" display="off"/>
+<attribute name="VALUE" x="-65.915" y="11.54" size="1.27" layer="27"/>
 </element>
 </elements>
@@
 <contactref element="R7" pad="1"/>
 <contactref element="PH1" pad="2"/>
-<wire x1="38.4" y1="1.7" x2="51.53" y2="10.24" width="0" layer="19" extent="1-1"/>
-<wire x1="57.27" y1="1.46" x2="38.4" y2="1.7" width="0" layer="19" extent="1-1"/>
-<wire x1="-31.99" y1="-2.54" x2="57.27" y2="1.46" width="0" layer="19" extent="1-1"/>
+<contactref element="R9" pad="1"/>
+<wire x1="-31.99" y1="-2.54" x2="-66.23" y2="8.96" width="0" layer="19" extent="1-1"/>
 <wire x1="-31.99" y1="0" x2="-31.99" y2="-2.54" width="0" layer="19" extent="1-1"/>
 <wire x1="-31.99" y1="2.54" x2="-31.99" y2="0" width="0" layer="19" extent="1-1"/>
@@
 <wire x1="3.85" y1="0" x2="-3.74" y2="0" width="0" layer="19" extent="1-1"/>
 <wire x1="16.896" y1="-9.9352" x2="3.85" y2="0" width="0" layer="19" extent="1-1"/>
+<wire x1="38.4" y1="1.7" x2="29.44" y2="-7.7" width="0" layer="19" extent="1-1"/>
+<wire x1="51.53" y1="10.24" x2="38.4" y2="1.7" width="0" layer="19" extent="1-1"/>
+<wire x1="57.27" y1="1.46" x2="51.53" y2="10.24" width="0" layer="19" extent="1-1"/>
 <wire x1="3.825" y1="-23.205" x2="16.896" y2="-9.9352" width="0" layer="19" extent="1-1"/>
 <wire x1="-3.425" y1="-22.555" x2="3.825" y2="-23.205" width="0" layer="19" extent="1-1"/>
@@
 <contactref element="R6" pad="1"/>
 <contactref element="R8" pad="2"/>
+<contactref element="R10" pad="2"/>
+<wire x1="55.37" y1="1.46" x2="-64.33" y2="14.08" width="0" layer="19" extent="1-1"/>
+<wire x1="59.21" y1="10.24" x2="55.37" y2="1.46" width="0" layer="19" extent="1-1"/>
+<wire x1="58.55" y1="16.64" x2="59.21" y2="10.24" width="0" layer="19" extent="1-1"/>
+</signal>
+<signal name="1V">
+<contactref element="R9" pad="2"/>
+<contactref element="R10" pad="1"/>
 <contactref element="IC1" pad="40"/>
-<wire x1="59.21" y1="10.24" x2="58.55" y2="16.64" width="0" layer="19" extent="1-1"/>
-<wire x1="55.37" y1="1.46" x2="59.21" y2="10.24" width="0" layer="19" extent="1-1"/>
-<wire x1="-2.12" y1="23.64" x2="58.55" y2="16.64" width="0" layer="19" extent="1-1"/>
+<wire x1="-66.23" y1="14.08" x2="-64.33" y2="8.96" width="0" layer="19" extent="1-1"/>
+<wire x1="-2.12" y1="23.64" x2="-66.23" y2="14.08" width="0" layer="19" extent="1-1"/>
 </signal>
 </signals>

Commit message: changed light Sensor to frequency Messurment
Parts:
- added C14, C15, C16: 100n, rcl:C0805
- added IC4: NE555D, linear:SO08
- added R11: 10k, rcl:R0805
- added R12: 33k, rcl:R0805
- R7: value 2k2 -> 1k
- R8: value 3k3 -> 10k
- moved R7 26.7 mm to (78.1, 17.9)
- moved R8 26.4 mm to (78.1, 0.00)
Connections:
- new net N$21: IC4.7, PH1.2, R7.1, R8.2
- new net N$22: C14.1, IC4.5
- new net N$23: C15.1, IC4.2, IC4.6, R7.2
- new net N$24: IC4.3, R11.2
- net +5V: now also C16.1, IC4.4, IC4.8, PH1.1, R8.1
- net 2.5V: no longer R8.2
- net GND: now also C14.2, C15.2, C16.2, IC4.1, R12.2; no longer PH1.2, R7.1
- net LIGHT: now also IC1.25, R11.1, R12.1; no longer IC1.41, PH1.1, R7.2, R8.1

Commit message: added lux messurment
Parts:
- added C17: 100n, rcl:C0805
Connections:
- net +5V: now also C17.1
- net N$21: now also C17.2
Changed lines of the file:
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@@
 <attribute name="VALUE" x="77.445" y="-15.34" size="1.27" layer="27"/>
+</element>
+<element name="C17" library="rcl" library_urn="urn:adsk.eagle:library:334" package="C0805" package3d_urn="urn:adsk.eagle:package:23617/2" value="100n" x="-96" y="-46.08" smashed="yes">
+<attribute name="NAME" x="-97.27" y="-44.81" size="1.27" layer="25"/>
+<attribute name="POPULARITY" value="88" x="-96" y="-46.08" size="1.778" layer="27" display="off"/>
+<attribute name="SPICEPREFIX" value="C" x="-96" y="-46.08" size="1.778" layer="27" display="off"/>
+<attribute name="VALUE" x="-97.27" y="-48.62" size="1.27" layer="27"/>
 </element>
 </elements>
@@
 <contactref element="C16" pad="1"/>
 <contactref element="R8" pad="1"/>
-<wire x1="77.13" y1="6.4" x2="77.13" y2="0" width="0" layer="19" extent="1-1"/>
-<wire x1="85.105" y1="3.8" x2="77.13" y2="6.4" width="0" layer="19" extent="1-1"/>
-<wire x1="81.295" y1="9" x2="85.105" y2="3.8" width="0" layer="19" extent="1-1"/>
-<wire x1="-66.36" y1="39.37" x2="81.295" y2="9" width="0" layer="19" extent="1-1"/>
+<contactref element="C17" pad="1"/>
+<wire x1="-14.946" y1="-27.31" x2="-96.95" y2="-46.08" width="0" layer="19" extent="1-1"/>
+<wire x1="-3.425" y1="-21.905" x2="-14.946" y2="-27.31" width="0" layer="19" extent="1-1"/>
+<wire x1="-6.28" y1="0" x2="-3.425" y2="-21.905" width="0" layer="19" extent="1-1"/>
+<wire x1="17.024" y1="-10.5448" x2="-3.425" y2="-21.905" width="0" layer="19" extent="1-1"/>
+<wire x1="38.4" y1="-1.7" x2="29.44" y2="-12.78" width="0" layer="19" extent="1-1"/>
+<wire x1="61.11" y1="10.24" x2="38.4" y2="-1.7" width="0" layer="19" extent="1-1"/>
+<wire x1="77.13" y1="6.4" x2="61.11" y2="10.24" width="0" layer="19" extent="1-1"/>
+<wire x1="81.295" y1="9" x2="77.13" y2="6.4" width="0" layer="19" extent="1-1"/>
+<wire x1="77.13" y1="0" x2="77.13" y2="6.4" width="0" layer="19" extent="1-1"/>
+<wire x1="85.105" y1="3.8" x2="81.295" y2="9" width="0" layer="19" extent="1-1"/>
+<wire x1="-66.36" y1="39.37" x2="-6.28" y2="0" width="0" layer="19" extent="1-1"/>
 <wire x1="-64.41" y1="48.26" x2="-66.36" y2="39.37" width="0" layer="19" extent="1-1"/>
 <wire x1="-58.06" y1="54.61" x2="-64.41" y2="48.26" width="0" layer="19" extent="1-1"/>
 <wire x1="-90.76" y1="59.69" x2="-64.41" y2="48.26" width="0" layer="19" extent="1-1"/>
-<wire x1="-6.28" y1="0" x2="-66.36" y2="39.37" width="0" layer="19" extent="1-1"/>
-<wire x1="-3.425" y1="-21.905" x2="-6.28" y2="0" width="0" layer="19" extent="1-1"/>
-<wire x1="-14.946" y1="-27.31" x2="-3.425" y2="-21.905" width="0" layer="19" extent="1-1"/>
-<wire x1="17.024" y1="-10.5448" x2="-3.425" y2="-21.905" width="0" layer="19" extent="1-1"/>
-<wire x1="38.4" y1="-1.7" x2="29.44" y2="-12.78" width="0" layer="19" extent="1-1"/>
-<wire x1="61.11" y1="10.24" x2="38.4" y2="-1.7" width="0" layer="19" extent="1-1"/>
 </signal>
 <signal name="D-">
@@
 <contactref element="R7" pad="1"/>
 <contactref element="R8" pad="2"/>
-<wire x1="77.13" y1="17.92" x2="79.03" y2="0" width="0" layer="19" extent="1-1"/>
-<wire x1="82.565" y1="9" x2="77.13" y2="17.92" width="0" layer="19" extent="1-1"/>
-<wire x1="38.4" y1="1.7" x2="82.565" y2="9" width="0" layer="19" extent="1-1"/>
+<contactref element="C17" pad="2"/>
+<wire x1="38.4" y1="1.7" x2="-95.05" y2="-46.08" width="0" layer="19" extent="1-1"/>
+<wire x1="79.03" y1="0" x2="38.4" y2="1.7" width="0" layer="19" extent="1-1"/>
+<wire x1="82.565" y1="9" x2="79.03" y2="0" width="0" layer="19" extent="1-1"/>
+<wire x1="77.13" y1="17.92" x2="82.565" y2="9" width="0" layer="19" extent="1-1"/>
 </signal>
 <signal name="N$22">
