File: biosphereMonitor.sch (EAGLE design)
At the start: 62 parts, among them IC1 XMEGA32A4AU, IC2 LM35, IC3 FT232RL, IC4 NE555D, IC5 SST25VF040, Q1 16Mhz, Q2 32kHz

Commit message: improved selftest
Parts:
- XIC6: value 78L05F -> 78L33
Changed lines of the file:
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@@
 <part name="+3V6" library="supply1" library_urn="urn:adsk.eagle:library:371" deviceset="+3V3" device=""/>
 <part name="C19" library="rcl" library_urn="urn:adsk.eagle:library:334" deviceset="CPOL-EU" device="G" package3d_urn="urn:adsk.eagle:package:23427/2" value="220µ"/>
-<part name="XIC6" library="linear" library_urn="urn:adsk.eagle:library:262" deviceset="78L*" device="F" package3d_urn="urn:adsk.eagle:package:16478/2" technology="05"/>
+<part name="XIC6" library="linear" library_urn="urn:adsk.eagle:library:262" deviceset="78L*" device="F" package3d_urn="urn:adsk.eagle:package:16478/2" technology="05" value="78L33"/>
 <part name="+3V12" library="supply1" library_urn="urn:adsk.eagle:library:371" deviceset="+3V3" device=""/>
 <part name="P+8" library="supply1" library_urn="urn:adsk.eagle:library:371" deviceset="+5V" device=""/>
